Commit message: added vi_sensor ro iris model and verified camera topics in ROS

File: models/rotors_description/urdf/iris_base.xacro (robot description, xacro)
@@ -11,5 +11,5 @@
   <xacro:arg name='enable_wind' default='false' />
   <!-- The following causes segfault with multiple vehicles if defaults to true!!! -->
-  <xacro:arg name='enable_ground_truth' default='false' />
+  <xacro:arg name='enable_ground_truth' default='true' />
   <xacro:arg name='enable_logging' default='false' />
   <xacro:arg name='log_file' default='iris' />
@@ -48,5 +48,5 @@
     mass_imu_sensor="0.015"
     gyroscope_noise_density="0.0003394"
-    gyroscopoe_random_walk="0.000038785"
+    gyroscope_random_walk="0.000038785"
     gyroscope_bias_correlation_time="1000.0"
     gyroscope_turn_on_bias_sigma="0.0087"
@@ -68,5 +68,5 @@
       mass_imu_sensor="0.00001"
       gyroscope_noise_density="0.0"
-      gyroscopoe_random_walk="0.0"
+      gyroscope_random_walk="0.0"
       gyroscope_bias_correlation_time="1000.0"
       gyroscope_turn_on_bias_sigma="0.0"
@@ -106,5 +106,5 @@
       image_scale=""
     >
-      <inertia ixx="0.00001" ixy="0.0" ixz="0.0" iyy="0.00001" iyz="0.0" izz="0.00001" /> <!-- [kg.m^2] [kg.m^2] [kg.m^2] [kg.m^2] [kg.m^2] [kg.m^2] -->
+      <inertia ixx="0.00001" ixy="0.0" ixz="0.0" iyy="0.00001" iyz="0.0" izz="0.00001" />
       <origin xyz="0.0 0.0 0.0" rpy="0.0 0.0 0.0" />
     </xacro:odometry_plugin_macro>
@@ -119,3 +119,32 @@
     </xacro:bag_plugin_macro>
   </xacro:if>
+<!--     <xacro:urock_odometry_plugin_macro
+    namespace="${namespace}"
+    odometry_sensor_suffix="1"
+    parent_link="base_link"
+    pose_topic="odometry_sensor1/pose"
+    pose_with_covariance_topic="odometry_sensor1/pose_with_covariance"
+    position_topic="odometry_sensor1/position"
+    transform_topic="odometry_sensor1/transform"
+    odometry_topic="odometry_sensor1/odometry"
+    parent_frame_id="world"
+    child_frame_id="odometry_sensor1"
+    mass_odometry_sensor="0.00001"
+    measurement_divisor="1"
+    measurement_delay="0"
+    unknown_delay="0.0"
+    noise_normal_position="0 0 0"
+    noise_normal_quaternion="0 0 0"
+    noise_normal_linear_velocity="0 0 0"
+    noise_normal_angular_velocity="0 0 0"
+    noise_uniform_position="0 0 0"
+    noise_uniform_quaternion="0 0 0"
+    noise_uniform_linear_velocity="0 0 0"
+    noise_uniform_angular_velocity="0 0 0"
+    enable_odometry_map="false"
+    odometry_map=""
+    image_scale="">
+    <inertia ixx="0.00001" ixy="0.0" ixz="0.0" iyy="0.00001" iyz="0.0" izz="0.00001" />
+    <origin xyz="0.0 0.0 0.0" rpy="0.0 0.0 0.0" />
+  </xacro:urock_odometry_plugin_macro> -->
 </robot>

Commit message: added opt flow cam (as vi_sensor model) to iris_base_vi_sensor

File: models/rotors_description/urdf/component_snippets.xacro (robot description, xacro)
@@ -17,4 +17,70 @@
 -->
 <robot xmlns:xacro="http://ros.org/wiki/xacro">
+    <!-- Optical Flow Camera Macro -->
+  <xacro:macro name="opt_flow_macro"
+    params="namespace parent_link *origin">
+    <link name="${namespace}/camera_opt_flow_link">
+      <collision>
+        <origin xyz="0 0 0" rpy="0 0 0" />
+        <geometry>
+          <box size="0.02 0.05 0.05" />
+        </geometry>
+      </collision>
+      <visual>
+        <origin xyz="0 0 0" rpy="0 0 0" />
+        <geometry>
+          <mesh filename="package://fastsense_description/meshes/vi_sensor.dae" scale="1 1 1" />
+        </geometry>
+      </visual>
+      <inertial>
+        <mass value="1e-5" />
+        <origin xyz="0 0 0" rpy="0 0 0" />
+        <inertia ixx="1e-6" ixy="0" ixz="0" iyy="1e-6" iyz="0" izz="1e-6" />
+      </inertial>
+    </link>
+    <joint name="${namespace}/camera_opt_flow_joint" type="fixed">
+      <xacro:insert_block name="origin" />
+      <parent link="${parent_link}" />
+      <child link="${namespace}/camera_opt_flow_link" />
+    </joint>
+    <gazebo reference="${namespace}/camera_opt_flow_link">
+      <sensor type="camera" name="${namespace}_camera_opt_flow">
+        <update_rate>20</update_rate>
+        <!-- <camera name="head"> -->
+        <camera>
+          <horizontal_fov>0.088</horizontal_fov>
+          <image>
+            <width>64</width>
+            <height>64</height>
+            <format>L8</format>
+          </image>
+          <clip>
+            <near>0.1</near>
+            <far>100</far>
+          </clip>
+          <noise>
+            <type>gaussian</type>
+            <mean>0.0</mean>
+            <stddev>0.001</stddev>
+          </noise>
+        </camera>
+        <plugin name="${namespace}_camera_opt_flow_controller" filename="libgazebo_opticalFlow_plugin.so">
+          <robotNamespace>${namespace}</robotNamespace>
+          <alwaysOn>true</alwaysOn>
+          <outputRate>20</outputRate>
+<!--           <cameraName>camera_${camera_suffix}</cameraName>
+          <imageTopicName>image_raw</imageTopicName>
+          <cameraInfoTopicName>camera_info</cameraInfoTopicName>
+          <frameName>camera_${camera_suffix}_link</frameName>
+          <hackBaseline>0.0</hackBaseline>
+          <distortionK1>0.0</distortionK1>
+          <distortionK2>0.0</distortionK2>
+          <distortionK3>0.0</distortionK3>
+          <distortionT1>0.0</distortionT1>
+          <distortionT2>0.0</distortionT2> -->
+        </plugin>
+      </sensor>
+    </gazebo>
+  </xacro:macro>
   <!-- Macro to add logging to a bag file. -->
   <xacro:macro name="bag_plugin_macro"

File: models/rotors_description/urdf/iris_base_vi_sensor.xacro (robot description, xacro)
@@ -12,5 +12,10 @@
 <!--     <mass value="0.00" />
     <inertia ixx="0.00000" ixy="0.0" ixz="0.0" iyy="0.00000" iyz="0.0" izz="0.00000" /> -->
-    <origin xyz="0.1 0.0 -0.03" rpy="0.0 0.1 0.0" />
+    <origin xyz="0.1 0.0 -0.03" rpy="0.0 0.0 0.0" />
   </xacro:vi_sensor_macro>
+  <xacro:opt_flow_macro
+    namespace="${namespace}/opt_flow_cam"
+    parent_link="base_link">
+    <origin xyz="0.0 0.0 -0.03" rpy="0.0 ${pi/2} 0.0" />
+  </xacro:opt_flow_macro>
 </robot>

Commit message: iris with opt flow and lidar urdf

File: models/rotors_description/urdf/component_snippets.xacro (robot description, xacro)
@@ -17,4 +17,122 @@
 -->
 <robot xmlns:xacro="http://ros.org/wiki/xacro">
+  <!-- Lidar Macro -->
+  <xacro:macro name="lidar_macro"
+    params="namespace parent_link *origin">
+    <link name="${namespace}/lidar_link">
+      <collision>
+        <origin xyz="0 0 0" rpy="0 0 0" />
+        <geometry>
+          <cylinder radius="0.06" length="0.05" />
+        </geometry>
+      </collision>
+      <visual>
+        <origin xyz="0 0 0" rpy="0 0 0" />
+        <geometry>
+          <cylinder radius="0.006" length="0.05" />
+        </geometry>
+      </visual>
+      <inertial>
+        <mass value="1e-5" />
+        <origin xyz="0 0 0" rpy="0 0 0" />
+        <inertia ixx="1e-6" ixy="0" ixz="0" iyy="1e-6" iyz="0" izz="1e-6" />
+      </inertial>
+    </link>
+    <joint name="${namespace}/lidar_joint" type="fixed">
+      <xacro:insert_block name="origin" />
+      <parent link="${parent_link}" />
+      <child link="${namespace}/lidar_link" />
+    </joint>
+    <gazebo reference="${namespace}/lidar_link">
+      <sensor type="ray" name="${namespace}_lidar">
+        <pose>0 0 0 0 -1.570896 0</pose>
+        <!-- <update_rate>20</update_rate> -->
+        <ray>
+          <scan>
+            <horizontal>
+              <samples>1</samples>
+              <resolution>1</resolution>
+              <min_angle>-0</min_angle>
+              <max_angle>0</max_angle>
+            </horizontal>
+          </scan>
+          <range>
+            <min>0.06</min>
+            <max>25</max>
+            <resolution>0.01</resolution>
+          </range>
+          <noise>
+            <type>gaussian</type>
+            <mean>0.0</mean>
+            <stddev>0.01</stddev>
+          </noise>
+        </ray>
+        <plugin name="${namespace}_lidar_controller" filename="libgazebo_lidar_plugin.so">
+          <robotNamespace>${namespace}</robotNamespace>
+          <always_on>1</always_on>
+          <update_rate>20</update_rate>
+          <visualize>true</visualize>
+        </plugin>
+      </sensor>
+    </gazebo>
+  </xacro:macro>
+    <!-- Optical Flow Camera Macro -->
+  <xacro:macro name="opt_flow_macro"
+    params="namespace parent_link *origin">
+    <link name="${namespace}/camera_opt_flow_link">
+      <collision>
+        <origin xyz="0 0 0" rpy="0 0 0" />
+        <geometry>
+          <box size="0.02 0.05 0.05" />
+        </geometry>
+      </collision>
+      <visual>
+        <origin xyz="0 0 0" rpy="0 0 0" />
+        <geometry>
+          <box size="0.02 0.05 0.05" />
+        </geometry>
+      </visual>
+      <inertial>
+        <mass value="1e-5" />
+        <origin xyz="0 0 0" rpy="0 0 0" />
+        <inertia ixx="1e-6" ixy="0" ixz="0" iyy="1e-6" iyz="0" izz="1e-6" />
+      </inertial>
+    </link>
+    <joint name="${namespace}/camera_opt_flow_joint" type="fixed">
+      <xacro:insert_block name="origin" />
+      <parent link="${parent_link}" />
+      <child link="${namespace}/camera_opt_flow_link" />
+    </joint>
+    <gazebo reference="${namespace}/camera_opt_flow_link">
+      <sensor type="camera" name="${namespace}_camera_opt_flow">
+        <always_on>true</always_on>
+        <update_rate>100.0</update_rate>
+        <visualize>true</visualize>
+        <topic>/px4flow</topic>
+        <camera>
+          <horizontal_fov>0.088</horizontal_fov>
+          <image>
+            <width>64</width>
+            <height>64</height>
+            <format>L8</format>
+          </image>
+          <clip>
+            <near>0.1</near>
+            <far>100</far>
+          </clip>
+          <noise>
+            <type>gaussian</type>
+            <mean>0.0</mean>
+            <stddev>0.001</stddev>
+          </noise>
+        </camera>
+        <plugin name="${namespace}_camera_opt_flow_controller" filename="libgazebo_opticalFlow_plugin.so">
+            <robotNamespace></robotNamespace>
+            <outputRate>20</outputRate>
+            <alwaysOn>true</alwaysOn>
+        </plugin>
+      </sensor>
+    </gazebo>
+  </xacro:macro>
   <!-- Macro to add logging to a bag file. -->
   <xacro:macro name="bag_plugin_macro"

File: models/rotors_description/urdf/iris_base_vi_sensor.xacro (robot description, xacro)
@@ -10,7 +10,15 @@
     enable_depth="true"
     enable_ground_truth="true">
-<!--     <mass value="0.00" />
-    <inertia ixx="0.00000" ixy="0.0" ixz="0.0" iyy="0.00000" iyz="0.0" izz="0.00000" /> -->
     <origin xyz="0.1 0.0 -0.03" rpy="0.0 0.1 0.0" />
   </xacro:vi_sensor_macro>
+  <xacro:opt_flow_macro
+    namespace="${namespace}/opt_flow_cam"
+    parent_link="base_link">
+    <origin xyz="-0.12 0.05 0.0" rpy="0.0 ${pi/2} ${pi/2}" />
+  </xacro:opt_flow_macro>
+  <xacro:lidar_macro
+    namespace="${namespace}/lidar"
+    parent_link="base_link">
+    <origin xyz="-0.12 0.0 0.0" rpy="0.0 ${pi} 0.0" />
+  </xacro:lidar_macro>
 </robot>
