Commit message: added vi_sensor meshes, updated xacro files to launch iris with opt flow and vi_sensor

File: models/rotors_description/urdf/component_snippets.xacro (robot description, xacro)
@@ -17,8 +17,7 @@
 -->
 <robot xmlns:xacro="http://ros.org/wiki/xacro">
-  <!-- Lidar Macro -->
   <xacro:macro name="lidar_macro"
-    params="namespace parent_link *origin">
-    <link name="${namespace}/lidar_link">
+    params="parent_link *origin">
+    <link name="lidar_link">
       <collision>
         <origin xyz="0 0 0" rpy="0 0 0" />
@@ -39,13 +38,15 @@
       </inertial>
     </link>
-    <joint name="${namespace}/lidar_joint" type="fixed">
+    <joint name="lidar_joint" type="revolute">
+      <parent link="${parent_link}" />
+      <child link="lidar_link" />
       <xacro:insert_block name="origin" />
-      <parent link="${parent_link}" />
-      <child link="${namespace}/lidar_link" />
-    </joint>
-    <gazebo reference="${namespace}/lidar_link">
-      <sensor type="ray" name="${namespace}_lidar">
-        <pose>0 0 0 0 -1.570896 0</pose>
-        <!-- <update_rate>20</update_rate> -->
+      <axis xyz="0 0 1"/>
+      <limit upper="0" lower="0" effort="-1" velocity="-1" />
+    </joint>
+    <gazebo reference="lidar_link">
+      <sensor type="ray" name="laser">
+        <pose>0 0 0 0 1.570896 0</pose>
+        <visualize>true</visualize>
         <ray>
           <scan>
@@ -68,14 +69,12 @@
           </noise>
         </ray>
-        <plugin name="${namespace}_lidar_controller" filename="libgazebo_lidar_plugin.so">
-          <robotNamespace>${namespace}</robotNamespace>
+        <plugin name="LaserPlugin" filename="libgazebo_lidar_plugin.so">
+          <robotNamespace></robotNamespace>
           <always_on>1</always_on>
           <update_rate>20</update_rate>
-          <visualize>true</visualize>
         </plugin>
       </sensor>
     </gazebo>
   </xacro:macro>
-    <!-- Optical Flow Camera Macro -->
   <xacro:macro name="opt_flow_macro"
     params="namespace parent_link *origin">
@@ -99,11 +98,12 @@
       </inertial>
     </link>
-    <joint name="${namespace}/camera_opt_flow_joint" type="fixed">
+    <joint name="${namespace}/camera_opt_flow_joint" type="revolute">
       <xacro:insert_block name="origin" />
       <parent link="${parent_link}" />
       <child link="${namespace}/camera_opt_flow_link" />
+      <limit upper="0" lower="0" effort="0" velocity="0" />
     </joint>
     <gazebo reference="${namespace}/camera_opt_flow_link">
-      <sensor type="camera" name="${namespace}_camera_opt_flow">
+      <sensor type="camera" name="PX4Flow">
         <always_on>true</always_on>
         <update_rate>100.0</update_rate>
@@ -127,8 +127,7 @@
           </noise>
         </camera>
-        <plugin name="${namespace}_camera_opt_flow_controller" filename="libgazebo_opticalFlow_plugin.so">
+        <plugin name="opticalflow_plugin" filename="libgazebo_opticalFlow_plugin.so">
             <robotNamespace></robotNamespace>
             <outputRate>20</outputRate>
-            <alwaysOn>true</alwaysOn>
         </plugin>
       </sensor>
@@ -314,57 +313,4 @@
     </gazebo>
   </xacro:macro>
-<!-- Macro to add a generic odometry sensor. -->
-  <xacro:macro name="odometry_plugin_macro"
-    params="
-      namespace odometry_sensor_suffix parent_link pose_topic pose_with_covariance_topic
-      position_topic transform_topic odometry_topic parent_frame_id
-      mass_odometry_sensor measurement_divisor measurement_delay unknown_delay
-      noise_normal_position noise_normal_quaternion noise_normal_linear_velocity
-      noise_normal_angular_velocity noise_uniform_position
-      noise_uniform_quaternion noise_uniform_linear_velocity
-      noise_uniform_angular_velocity enable_odometry_map odometry_map
-      image_scale *inertia *origin">
-    <!-- odometry link -->
-    <link name="${namespace}/odometry_sensor${odometry_sensor_suffix}_link">
-      <inertial>
-        <xacro:insert_block name="inertia" />
-        <mass value="${mass_odometry_sensor}" />  <!-- [kg] -->
-      </inertial>
-    </link>
-    <!-- odometry joint -->
-    <joint name="${namespace}/odometry_sensor${odometry_sensor_suffix}_joint" type="revolute">
-      <parent link="${parent_link}" />
-      <xacro:insert_block name="origin" />
-      <child link="${namespace}/odometry_sensor${odometry_sensor_suffix}_link" />
-      <limit upper="0" lower="0" effort="0" velocity="0" />
-    </joint>
-    <gazebo>
-      <plugin filename="librotors_gazebo_odometry_plugin.so" name="odometry_sensor${odometry_sensor_suffix}">
-        <linkName>${namespace}/odometry_sensor${odometry_sensor_suffix}_link</linkName>
-        <robotNamespace>${namespace}</robotNamespace>
-        <poseTopic>${pose_topic}</poseTopic>
-        <poseWithCovarianceTopic>${pose_with_covariance_topic}</poseWithCovarianceTopic>
-        <positionTopic>${position_topic}</positionTopic>
-        <transformTopic>${transform_topic}</transformTopic>
-        <odometryTopic>${odometry_topic}</odometryTopic>
-        <parentFrameId>${parent_frame_id}</parentFrameId>  <!-- Use the scoped link name here. e.g. Model::link. -->
-        <measurementDivisor>${measurement_divisor}</measurementDivisor> <!-- only every (seq % measurementDivisor) == 0 measurement is published [int] -->
-        <measurementDelay>${measurement_delay}</measurementDelay> <!-- time that measurement gets held back before it's published in [simulation cycles (int)] -->
-        <unknownDelay>${unknown_delay}</unknownDelay> <!-- additional delay, that just gets added to the timestamp [s] -->
-        <noiseNormalPosition>${noise_normal_position}</noiseNormalPosition> <!-- standard deviation of additive white gaussian noise [m] -->
-        <noiseNormalQuaternion>${noise_normal_quaternion}</noiseNormalQuaternion> <!-- standard deviation white gaussian noise [rad]: q_m = q*quaternionFromSmallAngleApproximation(noiseNormalQ) -->
-        <noiseNormalLinearVelocity>${noise_normal_linear_velocity}</noiseNormalLinearVelocity> <!-- standard deviation of additive white gaussian noise [m/s] -->
-        <noiseNormalAngularVelocity>${noise_normal_angular_velocity}</noiseNormalAngularVelocity> <!-- standard deviation of additive white gaussian noise [rad/s] -->
-        <noiseUniformPosition>${noise_uniform_position}</noiseUniformPosition> <!-- symmetric bounds of uniform noise [m] -->
-        <noiseUniformQuaternion>${noise_uniform_quaternion}</noiseUniformQuaternion> <!-- symmetric bounds of uniform noise [rad], computation see above -->
-        <noiseUniformLinearVelocity>${noise_uniform_linear_velocity}</noiseUniformLinearVelocity>  <!-- symmetric bounds of uniform noise [m/s] -->
-        <noiseUniformAngularVelocity>${noise_uniform_angular_velocity}</noiseUniformAngularVelocity>  <!-- symmetric bounds of uniform noise [rad/s] -->
-        <xacro:if value="${enable_odometry_map}">
-          <covarianceImage>package://rotors_gazebo/resource/${odometry_map}</covarianceImage>
-          <covarianceImageScale>${image_scale}</covarianceImageScale>
-        </xacro:if>
-      </plugin>
-    </gazebo>
-  </xacro:macro>
   <!-- Macro to add the wind plugin. -->
   <xacro:macro name="wind_plugin_macro"
@@ -717,17 +663,12 @@
         <origin xyz="0 0 0" rpy="0 0 0" />
         <geometry>
-          <mesh filename="package://fastsense_description/meshes/vi_sensor.dae" scale="1 1 1" />
+          <mesh filename="package://rotors_description/meshes/vi_sensor.dae" scale="1 1 1" />
         </geometry>
       </visual>
       <inertial>
-        <mass value="0.0" />
-        <origin xyz="0 0 0" rpy="0 0 0" />
-        <inertia ixx="0" ixy="0" ixz="0" iyy="0" iyz="0" izz="0" />
+        <mass value="0.13" />
+        <origin xyz="0 0 0" rpy="0 0 0" />
+        <inertia ixx="1e-6" ixy="0" ixz="0" iyy="1e-6" iyz="0" izz="1e-6" />
       </inertial>
-<!--   urock    <inertial>
-        <mass value="0.13" />
-        <origin xyz="0 0 0" rpy="0 0 0" />
-        <inertia ixx="1e-6" ixy="0" ixz="0" iyy="1e-6" iyz="0" izz="1e-6" />
-      </inertial>  -->
     </link>
     <joint name="${namespace}_vi_sensor_joint" type="fixed">
@@ -752,36 +693,4 @@
         <origin xyz="0.015 0.055 0.0065" rpy="0 0 0" />
       </xacro:vi_sensor_depth_macro>
-    </xacro:if>
-    <!-- Groundtruth -->
-    <xacro:if value="${enable_ground_truth}">
-      <!-- Odometry Sensor -->
-      <xacro:odometry_plugin_macro
-        namespace="${namespace}/ground_truth"
-        odometry_sensor_suffix=""
-        parent_link="${namespace}/vi_sensor_link"
-        pose_topic="pose"
-        pose_with_covariance_topic="pose_with_covariance"
-        position_topic="position"
-        transform_topic="transform"
-        odometry_topic="odometry"
-        parent_frame_id="world"
-        mass_odometry_sensor="0.00001"
-        measurement_divisor="1"
-        measurement_delay="0"
-        unknown_delay="0.0"
-        noise_normal_position="0 0 0"
-        noise_normal_quaternion="0 0 0"
-        noise_normal_linear_velocity="0 0 0"
-        noise_normal_angular_velocity="0 0 0"
-        noise_uniform_position="0 0 0"
-        noise_uniform_quaternion="0 0 0"
-        noise_uniform_linear_velocity="0 0 0"
-        noise_uniform_angular_velocity="0 0 0"
-        enable_odometry_map="false"
-        odometry_map=""
-        image_scale="">
-        <inertia ixx="0.00001" ixy="0.0" ixz="0.0" iyy="0.00001" iyz="0.0" izz="0.00001" /> <!-- [kg m^2] [kg m^2] [kg m^2] [kg m^2] [kg m^2] [kg m^2] -->
-        <origin xyz="0.0 0.0 0.0" rpy="0.0 0.0 0.0" />
-      </xacro:odometry_plugin_macro>
     </xacro:if>
     <!-- ADIS16448 IMU. -->

File: models/rotors_description/urdf/iris_base.xacro (robot description, xacro)
@@ -59,6 +59,7 @@
     <origin xyz="0 0 0" rpy="0 0 0" />
   </xacro:imu_plugin_macro>
+<!-- Mount an IMU providing ground truth. -->
+ <!-- Mount a generic odometry sensor providing ground truth. -->
   <xacro:if value="$(arg enable_ground_truth)">
-    <!-- Mount an IMU providing ground truth. -->
     <xacro:imu_plugin_macro
       namespace="${namespace}"
@@ -79,34 +80,4 @@
       <origin xyz="0 0 0" rpy="0 0 0" />
     </xacro:imu_plugin_macro>
-    <!-- Mount a generic odometry sensor providing ground truth. -->
-    <xacro:odometry_plugin_macro
-      namespace="${namespace}/ground_truth"
-      odometry_sensor_suffix="gt"
-      parent_link="base_link"
-      pose_topic="pose"
-      pose_with_covariance_topic="pose_with_covariance"
-      position_topic="position"
-      transform_topic="transform"
-      odometry_topic="odometry"
-      parent_frame_id="world"
-      mass_odometry_sensor="0.00001"
-      measurement_divisor="1"
-      measurement_delay="0"
-      unknown_delay="0.0"
-      noise_normal_position="0 0 0"
-      noise_normal_quaternion="0 0 0"
-      noise_normal_linear_velocity="0 0 0"
-      noise_normal_angular_velocity="0 0 0"
-      noise_uniform_position="0 0 0"
-      noise_uniform_quaternion="0 0 0"
-      noise_uniform_linear_velocity="0 0 0"
-      noise_uniform_angular_velocity="0 0 0"
-      enable_odometry_map="false"
-      odometry_map=""
-      image_scale=""
-    >
-      <inertia ixx="0.00001" ixy="0.0" ixz="0.0" iyy="0.00001" iyz="0.0" izz="0.00001" />
-      <origin xyz="0.0 0.0 0.0" rpy="0.0 0.0 0.0" />
-    </xacro:odometry_plugin_macro>
   </xacro:if>
   <xacro:if value="$(arg enable_logging)">
@@ -119,32 +90,3 @@
     </xacro:bag_plugin_macro>
   </xacro:if>
-<!--     <xacro:urock_odometry_plugin_macro
-    namespace="${namespace}"
-    odometry_sensor_suffix="1"
-    parent_link="base_link"
-    pose_topic="odometry_sensor1/pose"
-    pose_with_covariance_topic="odometry_sensor1/pose_with_covariance"
-    position_topic="odometry_sensor1/position"
-    transform_topic="odometry_sensor1/transform"
-    odometry_topic="odometry_sensor1/odometry"
-    parent_frame_id="world"
-    child_frame_id="odometry_sensor1"
-    mass_odometry_sensor="0.00001"
-    measurement_divisor="1"
-    measurement_delay="0"
-    unknown_delay="0.0"
-    noise_normal_position="0 0 0"
-    noise_normal_quaternion="0 0 0"
-    noise_normal_linear_velocity="0 0 0"
-    noise_normal_angular_velocity="0 0 0"
-    noise_uniform_position="0 0 0"
-    noise_uniform_quaternion="0 0 0"
-    noise_uniform_linear_velocity="0 0 0"
-    noise_uniform_angular_velocity="0 0 0"
-    enable_odometry_map="false"
-    odometry_map=""
-    image_scale="">
-    <inertia ixx="0.00001" ixy="0.0" ixz="0.0" iyy="0.00001" iyz="0.0" izz="0.00001" />
-    <origin xyz="0.0 0.0 0.0" rpy="0.0 0.0 0.0" />
-  </xacro:urock_odometry_plugin_macro> -->
 </robot>

File: models/rotors_description/urdf/iris_base_vi_sensor.xacro (robot description, xacro)
@@ -3,5 +3,4 @@
   <!-- Instantiate iris "mechanics" -->
   <xacro:include filename="$(arg rotors_description_dir)/urdf/iris_base.xacro" />
-  <!-- Mount a VI-sensor in front of the Firefly. -->
   <xacro:vi_sensor_macro
     namespace="${namespace}/vi_sensor"
@@ -13,12 +12,12 @@
   </xacro:vi_sensor_macro>
   <xacro:opt_flow_macro
-    namespace="${namespace}/opt_flow_cam"
+    namespace="${namespace}"
     parent_link="base_link">
     <origin xyz="-0.12 0.05 0.0" rpy="0.0 ${pi/2} ${pi/2}" />
   </xacro:opt_flow_macro>
   <xacro:lidar_macro
-    namespace="${namespace}/lidar"
     parent_link="base_link">
-    <origin xyz="-0.12 0.0 0.0" rpy="0.0 ${pi} 0.0" />
+    <!-- <origin xyz="-0.12 0.0 0.0" rpy="0.0 ${pi} 0.0" /> -->
+    <origin xyz="-0.12 0.0 0.0" rpy="0.0 0.0 0.0" />
   </xacro:lidar_macro>
 </robot>

File: models/rotors_description/urdf/multirotor_base.xacro (robot description, xacro)
@@ -35,5 +35,5 @@
         <origin xyz="0 0 0" rpy="0 0 0" />
         <geometry>
-          <mesh filename="package://fastsense_description/meshes/${mesh_file}"
+          <mesh filename="package://rotors_description/meshes/${mesh_file}"
             scale="${mesh_scale}" />
           <!-- <box size="${body_width} ${body_width} ${body_height}"/> --> <!-- [m] [m] [m] -->
@@ -55,4 +55,5 @@
       </plugin>
       <plugin name="ground_truth_pose" filename="libgazebo_ros_p3d.so">
+        <robotNamespace>${robot_namespace}</robotNamespace>
         <alwaysOn>true</alwaysOn>
         <updateRate>100.0</updateRate>
@@ -102,6 +103,6 @@
         <geometry>
           <!-- <cylinder length="0.005" radius="${radius_rotor}"/> --> <!-- [m] -->
-          <!-- <mesh filename="package://fastsense_description/meshes/propeller_${direction}.dae" -->
-          <mesh filename="package://fastsense_description/meshes/${mesh}_${direction}.dae"
+          <!-- <mesh filename="package://rotors_description/meshes/propeller_${direction}.dae" -->
+          <mesh filename="package://rotors_description/meshes/${mesh}_${direction}.dae"
             scale="${mesh_scale}" />
           <!-- <box size="${2*radius_rotor} 0.01 0.005"/> -->

Commit message: rename iris_base_vi_sensor.xacro -> iris_vi_sensor.xacro, deleted opt flow stuff from urdf

File: models/rotors_description/urdf/component_snippets.xacro (robot description, xacro)
@@ -17,121 +17,4 @@
 -->
 <robot xmlns:xacro="http://ros.org/wiki/xacro">
-  <xacro:macro name="lidar_macro"
-    params="parent_link *origin">
-    <link name="lidar_link">
-      <collision>
-        <origin xyz="0 0 0" rpy="0 0 0" />
-        <geometry>
-          <cylinder radius="0.06" length="0.05" />
-        </geometry>
-      </collision>
-      <visual>
-        <origin xyz="0 0 0" rpy="0 0 0" />
-        <geometry>
-          <cylinder radius="0.006" length="0.05" />
-        </geometry>
-      </visual>
-      <inertial>
-        <mass value="1e-5" />
-        <origin xyz="0 0 0" rpy="0 0 0" />
-        <inertia ixx="1e-6" ixy="0" ixz="0" iyy="1e-6" iyz="0" izz="1e-6" />
-      </inertial>
-    </link>
-    <joint name="lidar_joint" type="revolute">
-      <parent link="${parent_link}" />
-      <child link="lidar_link" />
-      <xacro:insert_block name="origin" />
-      <axis xyz="0 0 1"/>
-      <limit upper="0" lower="0" effort="-1" velocity="-1" />
-    </joint>
-    <gazebo reference="lidar_link">
-      <sensor type="ray" name="laser">
-        <pose>0 0 0 0 1.570896 0</pose>
-        <visualize>true</visualize>
-        <ray>
-          <scan>
-            <horizontal>
-              <samples>1</samples>
-              <resolution>1</resolution>
-              <min_angle>-0</min_angle>
-              <max_angle>0</max_angle>
-            </horizontal>
-          </scan>
-          <range>
-            <min>0.06</min>
-            <max>25</max>
-            <resolution>0.01</resolution>
-          </range>
-          <noise>
-            <type>gaussian</type>
-            <mean>0.0</mean>
-            <stddev>0.01</stddev>
-          </noise>
-        </ray>
-        <plugin name="LaserPlugin" filename="libgazebo_lidar_plugin.so">
-          <robotNamespace></robotNamespace>
-          <always_on>1</always_on>
-          <update_rate>20</update_rate>
-        </plugin>
-      </sensor>
-    </gazebo>
-  </xacro:macro>
-  <xacro:macro name="opt_flow_macro"
-    params="namespace parent_link *origin">
-    <link name="${namespace}/camera_opt_flow_link">
-      <collision>
-        <origin xyz="0 0 0" rpy="0 0 0" />
-        <geometry>
-          <box size="0.02 0.05 0.05" />
-        </geometry>
-      </collision>
-      <visual>
-        <origin xyz="0 0 0" rpy="0 0 0" />
-        <geometry>
-          <box size="0.02 0.05 0.05" />
-        </geometry>
-      </visual>
-      <inertial>
-        <mass value="1e-5" />
-        <origin xyz="0 0 0" rpy="0 0 0" />
-        <inertia ixx="1e-6" ixy="0" ixz="0" iyy="1e-6" iyz="0" izz="1e-6" />
-      </inertial>
-    </link>
-    <joint name="${namespace}/camera_opt_flow_joint" type="revolute">
-      <xacro:insert_block name="origin" />
-      <parent link="${parent_link}" />
-      <child link="${namespace}/camera_opt_flow_link" />
-      <limit upper="0" lower="0" effort="0" velocity="0" />
-    </joint>
-    <gazebo reference="${namespace}/camera_opt_flow_link">
-      <sensor type="camera" name="PX4Flow">
-        <always_on>true</always_on>
-        <update_rate>100.0</update_rate>
-        <visualize>true</visualize>
-        <topic>/px4flow</topic>
-        <camera>
-          <horizontal_fov>0.088</horizontal_fov>
-          <image>
-            <width>64</width>
-            <height>64</height>
-            <format>L8</format>
-          </image>
-          <clip>
-            <near>0.1</near>
-            <far>100</far>
-          </clip>
-          <noise>
-            <type>gaussian</type>
-            <mean>0.0</mean>
-            <stddev>0.001</stddev>
-          </noise>
-        </camera>
-        <plugin name="opticalflow_plugin" filename="libgazebo_opticalFlow_plugin.so">
-            <robotNamespace></robotNamespace>
-            <outputRate>20</outputRate>
-        </plugin>
-      </sensor>
-    </gazebo>
-  </xacro:macro>
   <!-- Macro to add logging to a bag file. -->
   <xacro:macro name="bag_plugin_macro"

File: models/rotors_description/urdf/iris_vi_sensor.xacro (robot description, xacro)
@@ -11,13 +11,3 @@
     <origin xyz="0.1 0.0 -0.03" rpy="0.0 0.1 0.0" />
   </xacro:vi_sensor_macro>
-  <xacro:opt_flow_macro
-    namespace="${namespace}"
-    parent_link="base_link">
-    <origin xyz="-0.12 0.05 0.0" rpy="0.0 ${pi/2} ${pi/2}" />
-  </xacro:opt_flow_macro>
-  <xacro:lidar_macro
-    parent_link="base_link">
-    <!-- <origin xyz="-0.12 0.0 0.0" rpy="0.0 ${pi} 0.0" /> -->
-    <origin xyz="-0.12 0.0 0.0" rpy="0.0 0.0 0.0" />
-  </xacro:lidar_macro>
 </robot>

Commit message: removed depth sensor from vi_sensor urdf, set camera frame rate = 15 fps

File: models/rotors_description/urdf/component_snippets.xacro (robot description, xacro)
@@ -544,5 +544,5 @@
   </xacro:macro>
   <!-- VI-Sensor Macro -->
-  <xacro:macro name="vi_sensor_macro" params="namespace parent_link enable_cameras enable_depth enable_ground_truth *origin">
+  <xacro:macro name="vi_sensor_macro" params="namespace parent_link enable_cameras frame_rate enable_depth enable_ground_truth *origin">
     <!-- Vi Sensor Link -->
     <link name="${namespace}/vi_sensor_link">
@@ -575,5 +575,5 @@
       <xacro:vi_sensor_stereo_camera_macro
         namespace="${namespace}" parent_link="${namespace}/vi_sensor_link"
-        frame_rate="30.0" origin_offset_x="0.015" baseline_y="${0.055*2}"
+        frame_rate="${frame_rate}" origin_offset_x="0.015" baseline_y="${0.055*2}"
         origin_offset_z="0.0065" max_range="30.0">
       </xacro:vi_sensor_stereo_camera_macro>

File: models/rotors_description/urdf/iris_vi_sensor.xacro (robot description, xacro)
@@ -7,5 +7,6 @@
     parent_link="base_link"
     enable_cameras="true"
-    enable_depth="true"
+    frame_rate="15"
+    enable_depth="false"
     enable_ground_truth="true">
     <origin xyz="0.1 0.0 -0.03" rpy="0.0 0.1 0.0" />

Commit message: changed depth camera params to match rgb camera fov and matrix

File: models/rotors_description/urdf/component_snippets.xacro (robot description, xacro)
@@ -381,4 +381,5 @@
     <joint name="${namespace}/camera_${camera_suffix}_optical_center_joint" type="fixed">
       <origin xyz="0 0 0" rpy="${-pi/2} 0 ${-pi/2}" />
+      <!-- <origin xyz="0 0 0" rpy="0 0 0" /> -->
       <parent link="${namespace}/camera_${camera_suffix}_link" />
       <child link="${namespace}/camera_${camera_suffix}_optical_center_link" />
@@ -390,8 +391,11 @@
         <update_rate>${frame_rate}</update_rate>
         <camera>
-          <horizontal_fov>2</horizontal_fov>
+          <!-- <horizontal_fov>2</horizontal_fov> -->
+          <horizontal_fov>1.3962634</horizontal_fov>
           <image>
             <format>R8G8B8</format>
-            <width>640</width>
+<!--             <width>640</width>
+            <height>480</height> -->
+            <width>752</width>
             <height>480</height>
           </image>
@@ -583,5 +587,5 @@
       <xacro:vi_sensor_depth_macro
         namespace="${namespace}" parent_link="${namespace}/vi_sensor_link"
-        camera_suffix="depth" frame_rate="30.0" max_range="10.0">
+        camera_suffix="depth" frame_rate="${frame_rate}" max_range="10.0">
         <origin xyz="0.015 0.055 0.0065" rpy="0 0 0" />
       </xacro:vi_sensor_depth_macro>

File: models/rotors_description/urdf/iris_vi_sensor.xacro (robot description, xacro)
@@ -7,8 +7,9 @@
     parent_link="base_link"
     enable_cameras="true"
-    frame_rate="15"
-    enable_depth="false"
+    frame_rate="20"
+    enable_depth="true"
     enable_ground_truth="true">
-    <origin xyz="0.1 0.0 -0.03" rpy="0.0 0.1 0.0" />
+    <!-- <origin xyz="0.1 0.0 -0.03" rpy="0.0 0.1 0.0" /> -->
+    <origin xyz="0.1 0.0 -0.03" rpy="0.0 0.0 0.0" />
   </xacro:vi_sensor_macro>
 </robot>
